Commit message: adjusting some more the demonstration

File: src/sorting_demo/models/block/block.urdf.xacro (robot description, xacro)
@@ -4,20 +4,20 @@
   <link name="block">
     <inertial>
-      <origin xyz="0.025 0.025 0.025" />
-      <mass value="0.5" />
+      <origin xyz="0.02 0.02 0.02" />
+      <mass value="0.25" />
       <!-- (1/12)*mass*(h^2 + d^2)  (1/12)*mass*(w^2 + d^2) (1/12)*mass*(w^2 + h^2) -->
-      <!-- (1/12)*0.5*(0.045^2 + 0.045^2)  (1/12)*0.5*(0.045^2 + 0.045^2) (1/12)*0.5*(0.045^2 + 0.045^2) -->
+      <!-- (1/12)*0.5*(0.04^2 + 0.04^2)  (1/12)*0.5*(0.04^2 + 0.04^2) (1/12)*0.5*(0.04^2 + 0.04^2) -->
       <inertia  ixx="0.00016874999" ixy="0.0"  ixz="0.0"  iyy="0.00016874999"  iyz="0.0"  izz="0.00016874999" />
     </inertial>
     <visual>
-      <origin xyz="0.025 0.025 0.025"/>
+      <origin xyz="0.02 0.02 0.02"/>
       <geometry>
-        <box size="0.045 0.045 0.045" />
+        <box size="0.04 0.04 0.04" />
       </geometry>
     </visual>
     <collision>
-      <origin xyz="0.025 0.025 0.025"/>
+      <origin xyz="0.02 0.02 0.02"/>
       <geometry>
-        <box size="0.045 0.045 0.045" />
+        <box size="0.04 0.04 0.04" />
       </geometry>
     </collision>

Commit message: torsional friction for blocks

File: src/sorting_demo/models/block/block.urdf.xacro (robot description, xacro)
@@ -8,5 +8,5 @@
       <!-- (1/12)*mass*(h^2 + d^2)  (1/12)*mass*(w^2 + d^2) (1/12)*mass*(w^2 + h^2) -->
       <!-- (1/12)*0.5*(0.04^2 + 0.04^2)  (1/12)*0.5*(0.04^2 + 0.04^2) (1/12)*0.5*(0.04^2 + 0.04^2) -->
-      <inertia  ixx="0.00016874999" ixy="0.0"  ixz="0.0"  iyy="0.00016874999"  iyz="0.0"  izz="0.00016874999" />
+      <inertia  ixx="0.000066667" ixy="0.0"  ixz="0.0"  iyy="0.000066667"  iyz="0.0"  izz="0.000066667" />
     </inertial>
     <visual>
@@ -25,6 +25,17 @@
   <gazebo reference="block">
      <material>$(arg material)</material>
-     <mu1>1000</mu1>
-     <mu2>1000</mu2>
+     <mu1>10000</mu1>
+     <mu2>10000</mu2>
+  <collision>
+      <surface>
+        <friction>
+          <torsional>
+            <coefficient>0.456</coefficient>
+            <use_patch_radius>true</use_patch_radius>
+            <patch_radius>0.05</patch_radius>
+          </torsional>
+        </friction>
+      </surface>
+    </collision>
   </gazebo>
 </robot>

Commit message: Minor changes in the block description

File: src/sorting_demo/models/block/block.urdf.xacro (robot description, xacro)
@@ -2,22 +2,21 @@
        name="block">
   <xacro:arg name="material" default="Gazebo/Black" />
+  <xacro:arg name="edge_length" default="0.04" />
+  <xacro:property name="block_density" value="3900" />
   <link name="block">
     <inertial>
-      <origin xyz="0.02 0.02 0.02" />
-      <mass value="0.25" />
-      <!-- (1/12)*mass*(h^2 + d^2)  (1/12)*mass*(w^2 + d^2) (1/12)*mass*(w^2 + h^2) -->
-      <!-- (1/12)*0.5*(0.04^2 + 0.04^2)  (1/12)*0.5*(0.04^2 + 0.04^2) (1/12)*0.5*(0.04^2 + 0.04^2) -->
-      <inertia  ixx="0.000066667" ixy="0.0"  ixz="0.0"  iyy="0.000066667"  iyz="0.0"  izz="0.000066667" />
+      <mass value="${block_density * $(arg edge_length)**3}" />
+      <inertia  ixx="${(1/12) * block_density * $(arg edge_length)**3 * (2 * $(arg edge_length)**2)}" ixy="0.0" ixz="0.0"
+                iyy="${(1/12) * block_density * $(arg edge_length)**3 * (2 * $(arg edge_length)**2)}" iyz="0.0"
+                izz="${(1/12) * block_density * $(arg edge_length)**3 * (2 * $(arg edge_length)**2)}" />
     </inertial>
     <visual>
-      <origin xyz="0.02 0.02 0.02"/>
       <geometry>
-        <box size="0.04 0.04 0.04" />
+        <box size="$(arg edge_length) $(arg edge_length) $(arg edge_length)" />
       </geometry>
     </visual>
     <collision>
-      <origin xyz="0.02 0.02 0.02"/>
       <geometry>
-        <box size="0.04 0.04 0.04" />
+        <box size="$(arg edge_length) $(arg edge_length) $(arg edge_length)" />
       </geometry>
     </collision>
