Commit message: a bit more thicker tray

File: src/sorting_demo/models/tray/tray.urdf.xacro (robot description, xacro)
@@ -3,5 +3,5 @@
   <xacro:property name="tray_length" value="0.3" />
   <xacro:property name="tray_height" value="0.05" />
-  <xacro:property name="tray_thickness" value="0.01" />
+  <xacro:property name="tray_thickness" value="0.015" />
   <xacro:property name="tray_density" value="950" />
   <xacro:property name="tray_base_name" value="tray_base" />

Commit message: more work on tray picking

File: src/sorting_demo/models/tray/tray.urdf.xacro (robot description, xacro)
@@ -29,4 +29,15 @@
        <mu1>1000</mu1>
        <mu2>1000</mu2>
+      <collision>
+          <surface>
+            <friction>
+              <torsional>
+                <coefficient>0.456</coefficient>
+                <use_patch_radius>true</use_patch_radius>
+                <patch_radius>0.05</patch_radius>
+              </torsional>
+            </friction>
+          </surface>
+        </collision>
     </gazebo>
     <xacro:if value="${xPos != 0 or yPos != 0}">
@@ -38,8 +49,8 @@
     </xacro:if>
   </xacro:macro>
-  <xacro:tray_part name="${tray_base_name}" width="${tray_width}" length="${tray_length}" height="${tray_thickness}" mass="0.5" material="Gazebo/White" />
-  <xacro:tray_part name="tray_wall0" width="${tray_width - 2 * tray_thickness}" length="${tray_thickness}" height="${tray_height}" mass="0.1" material="Gazebo/Red" yPos="-1" />
-  <xacro:tray_part name="tray_wall1" width="${tray_width - 2 * tray_thickness}" length="${tray_thickness}" height="${tray_height}" mass="0.1" material="Gazebo/Red" yPos="1" />
-  <xacro:tray_part name="tray_wall2" width="${tray_thickness}" length="${tray_length}" height="${tray_height}" mass="0.1" material="Gazebo/Blue" xPos="-1" />
-  <xacro:tray_part name="tray_wall3" width="${tray_thickness}" length="${tray_length}" height="${tray_height}" mass="0.1" material="Gazebo/Blue" xPos="1" />
+  <xacro:tray_part name="${tray_base_name}" width="${tray_width}" length="${tray_length}" height="${tray_thickness}" mass="0.05" material="Gazebo/White" />
+  <xacro:tray_part name="tray_wall0" width="${tray_width - 2 * tray_thickness}" length="${tray_thickness}" height="${tray_height}" mass="0.01" material="Gazebo/Red" yPos="-1" />
+  <xacro:tray_part name="tray_wall1" width="${tray_width - 2 * tray_thickness}" length="${tray_thickness}" height="${tray_height}" mass="0.01" material="Gazebo/Red" yPos="1" />
+  <xacro:tray_part name="tray_wall2" width="${tray_thickness}" length="${tray_length}" height="${tray_height}" mass="0.01" material="Gazebo/Blue" xPos="-1" />
+  <xacro:tray_part name="tray_wall3" width="${tray_thickness}" length="${tray_length}" height="${tray_height}" mass="0.01" material="Gazebo/Blue" xPos="1" />
 </robot>

Commit message: moving pieces one by one from trays to tabletop

File: src/sorting_demo/models/tray/tray.urdf.xacro (robot description, xacro)
@@ -1,7 +1,7 @@
 <robot xmlns:xacro="http://ros.org/wiki/xacro" name="tray">
   <xacro:property name="tray_width" value="0.2" />
-  <xacro:property name="tray_length" value="0.3" />
+  <xacro:property name="tray_length" value="0.32" />
   <xacro:property name="tray_height" value="0.05" />
-  <xacro:property name="tray_thickness" value="0.015" />
+  <xacro:property name="tray_thickness" value="0.01" />
   <xacro:property name="tray_density" value="950" />
   <xacro:property name="tray_base_name" value="tray_base" />

Commit message: updating repositories submodules to intera 5.3 and other minor changes

File: src/sorting_demo/models/tray/tray.urdf.xacro (robot description, xacro)
@@ -3,6 +3,6 @@
   <xacro:property name="tray_length" value="0.32" />
   <xacro:property name="tray_height" value="0.05" />
-  <xacro:property name="tray_thickness" value="0.01" />
-  <xacro:property name="tray_density" value="950" />
+  <xacro:property name="tray_thickness" value="0.015" />
+  <xacro:property name="tray_density" value="100" />
   <xacro:property name="tray_base_name" value="tray_base" />
   <xacro:macro name="tray_part" params="name width length height mass material xPos:=0 yPos:=0">
@@ -49,5 +49,5 @@
     </xacro:if>
   </xacro:macro>
-  <xacro:tray_part name="${tray_base_name}" width="${tray_width}" length="${tray_length}" height="${tray_thickness}" mass="0.05" material="Gazebo/White" />
+  <xacro:tray_part name="${tray_base_name}" width="${tray_width}" length="${tray_length}" height="${tray_thickness}" mass="0.01" material="Gazebo/White" />
   <xacro:tray_part name="tray_wall0" width="${tray_width - 2 * tray_thickness}" length="${tray_thickness}" height="${tray_height}" mass="0.01" material="Gazebo/Red" yPos="-1" />
   <xacro:tray_part name="tray_wall1" width="${tray_width - 2 * tray_thickness}" length="${tray_thickness}" height="${tray_height}" mass="0.01" material="Gazebo/Red" yPos="1" />

Commit message: more optimized and safe simulation

File: src/sorting_demo/models/tray/tray.urdf.xacro (robot description, xacro)
@@ -9,5 +9,5 @@
     <link name="${name}">
       <inertial>
-        <mass value="${tray_density * width * length * height}" />
+        <mass value="${tray_density * width * length * height*1000.0}" />
         <inertia  ixx="${(1/12) * tray_density * width * length * height * (length**2 + height**2)}" ixy="0.0"  ixz="0.0"
                   iyy="${(1/12) * tray_density * width * length * height * (width**2 + height**2)}"  iyz="0.0"
@@ -40,5 +40,7 @@
           </surface>
         </collision>
-        <is_static>true</is_static>
+    </gazebo>
+    <gazebo reference="$tray">
+        <static>true</static>
     </gazebo>
     <xacro:if value="${xPos != 0 or yPos != 0}">

Commit message: White tray

File: src/sorting_demo/models/tray/tray.urdf.xacro (robot description, xacro)
@@ -9,5 +9,5 @@
     <link name="${name}">
       <inertial>
-        <mass value="${tray_density * width * length * height*1000.0}" />
+        <mass value="${tray_density * width * length * height}" />
         <inertia  ixx="${(1/12) * tray_density * width * length * height * (length**2 + height**2)}" ixy="0.0"  ixz="0.0"
                   iyy="${(1/12) * tray_density * width * length * height * (width**2 + height**2)}"  iyz="0.0"
@@ -41,5 +41,5 @@
         </collision>
     </gazebo>
-    <gazebo reference="$tray">
+    <gazebo>
         <static>true</static>
     </gazebo>
@@ -53,7 +53,7 @@
   </xacro:macro>
   <xacro:tray_part name="${tray_base_name}" width="${tray_width}" length="${tray_length}" height="${tray_thickness}" mass="0.01" material="Gazebo/White" />
-  <xacro:tray_part name="tray_wall0" width="${tray_width - 2 * tray_thickness}" length="${tray_thickness}" height="${tray_height}" mass="0.01" material="Gazebo/Red" yPos="-1" />
-  <xacro:tray_part name="tray_wall1" width="${tray_width - 2 * tray_thickness}" length="${tray_thickness}" height="${tray_height}" mass="0.01" material="Gazebo/Red" yPos="1" />
-  <xacro:tray_part name="tray_wall2" width="${tray_thickness}" length="${tray_length}" height="${tray_height}" mass="0.01" material="Gazebo/Blue" xPos="-1" />
-  <xacro:tray_part name="tray_wall3" width="${tray_thickness}" length="${tray_length}" height="${tray_height}" mass="0.01" material="Gazebo/Blue" xPos="1" />
+  <xacro:tray_part name="tray_wall0" width="${tray_width - 2 * tray_thickness}" length="${tray_thickness}" height="${tray_height}" mass="0.01" material="Gazebo/White" yPos="-1" />
+  <xacro:tray_part name="tray_wall1" width="${tray_width - 2 * tray_thickness}" length="${tray_thickness}" height="${tray_height}" mass="0.01" material="Gazebo/White" yPos="1" />
+  <xacro:tray_part name="tray_wall2" width="${tray_thickness}" length="${tray_length}" height="${tray_height}" mass="0.01" material="Gazebo/White" xPos="-1" />
+  <xacro:tray_part name="tray_wall3" width="${tray_thickness}" length="${tray_length}" height="${tray_height}" mass="0.01" material="Gazebo/White" xPos="1" />
 </robot>
